Commit message: loading model done

File: models/wam_top.urdf.xacro (robot description, xacro)
@@ -12,4 +12,6 @@
   <!-- Definitions for the barrett ball -->
   <xacro:include filename="$(find barrett_model)/models/ball.urdf.xacro"/>
+  <!-- Definitions for the table and cube -->
+  <xacro:include filename="$(find barrett_model)/robots/table.urdf.xacro"/>
   <!-- Materials -->
   <material name="WAMGrey">

File: robots/table.urdf (robot description, URDF)
Before this commit: robot table_no_wheels, 1 links, 0 joints
Links:
- removed link table
- added link base_link; visual box size=0.83 0.70 0.05
- added link cube; visual box size=0.08 0.08 0.08
Joints:
- added joint scene: type fixed, parent base_link, child cube

File: robots/table.urdf.xacro (robot description, xacro)
@@ -1,15 +1,41 @@
-<?xml version="1.0" ?>
+<?xml version="1.0"?>
 <!-- =================================================================================== -->
 <!-- |    This document was autogenerated by xacro from table.urdf                     | -->
 <!-- |    EDITING THIS FILE BY HAND IS NOT RECOMMENDED                                 | -->
 <!-- =================================================================================== -->
-<robot name="table">
-  <link name="table">
-    <visual>
-      <origin rpy="0 0 0" xyz="0 0.5 0"/>
-      <geometry>
-        <mesh filename="package://barrett_model/models/object_meshes/table_no_wheels.dae"/>
-      </geometry>
-    </visual>
-  </link>
+<robot xmlns:xacro="http://ros.org/wiki/xacro">
+  <xacro:macro name="table" params="prefix parent_link xyz rpy">
+    <link name="table_top">
+      <visual>
+        <material name="table_color">
+          <color rgba="0.0 0.5 0.5 1.0"/>
+        </material>
+        <geometry>
+          <box size="0.83 0.70 0.05"/>
+        </geometry>
+      </visual>
+    </link>
+    <joint name="table" type="fixed">
+      <parent link="${parent_link}"/>
+      <child link="table_top"/>
+      <origin xyz="${xyz}" rpy="${rpy}"/>
+    </joint>
+  </xacro:macro>
+  <xacro:macro name="cube" params="prefix parent_link xyz rpy">
+    <link name="cube_08">
+      <visual>
+        <material name="cube_color">
+          <color rgba="0.01 0.1 0.1 1.0"/>
+        </material>
+        <geometry>
+          <box size="0.08 0.08 0.08"/>
+        </geometry>
+      </visual>
+    </link>
+    <joint name="cube" type="fixed">
+      <parent link="${parent_link}"/>
+      <child link="cube_08"/>
+      <origin xyz="${xyz}" rpy="${rpy}"/>
+    </joint>
+  </xacro:macro>
 </robot>

File: robots/wam_7dof_wam_bhand.urdf.xacro (robot description, xacro)
@@ -7,3 +7,5 @@
   <xacro:wam_7dof prefix="wam" parent_link="world" xyz="0 0 0" rpy="0 0 0" />
   <xacro:bhand prefix="wam/bhand" parent_link="wam/wrist_palm_link" xyz="0 0 0.06" rpy="0 0 ${PI}"/>
+  <xacro:table prefix="table" parent_link="world" xyz="0.9 0 0.5" rpy="0 0 0"/>
+  <xacro:cube prefix="cube" parent_link="world" xyz="0.9 0 0.565" rpy="0 0 0"/>
 </robot>
