Commit message: making changes

File: robots/table.urdf.xacro (robot description, xacro)
@@ -12,5 +12,5 @@
         </material>
         <geometry>
-          <box size="0.83 0.70 0.05"/>
+          <box size="0.775 0.83 0.05"/>
         </geometry>
       </visual>

File: robots/wam_7dof_wam_bhand.urdf.xacro (robot description, xacro)
@@ -5,7 +5,7 @@
   <!-- Root link is in the world frame-->
   <link name = "world"/>
-  <xacro:wam_7dof prefix="wam" parent_link="world" xyz="0 0 0" rpy="0 0 0" />
-  <xacro:bhand prefix="wam/bhand" parent_link="wam/wrist_palm_link" xyz="0 0 0.06" rpy="0 0 ${PI}"/>
-  <xacro:table prefix="table" parent_link="world" xyz="0.9 0 0.5" rpy="0 0 0"/>
-  <xacro:cube prefix="cube" parent_link="world" xyz="0.9 0 0.565" rpy="0 0 0"/>
+  <xacro:wam_7dof prefix="wam" parent_link="world" xyz="0 0 0.70" rpy="0 0 -1.5708" />
+  <xacro:bhand prefix="wam/bhand" parent_link="wam/wrist_palm_link" xyz="0 0 0.06" rpy="0 0 0"/>
+  <xacro:table prefix="table" parent_link="world" xyz="0.7175 0 0.725" rpy="0 0 0"/>
+  <xacro:cube prefix="cube" parent_link="world" xyz="0.7175 0 0.79" rpy="0 0 0"/>
 </robot>
